File: THS-80.kicad_pcb (KiCad board)
At the start: 4 copper layers, 101.6 x 102.1 mm, 120 parts, among them J1 USB_B_Micro, J10 PIO Header, J2 RC80 Bus, J3 RC80 Expansion, J4 JTAG, J5 PMOD, J6 CT0, J7 Port A, J8 Port A, J9 IDE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

Commit message: started routing
Parts:
- R21, R23, R24, R25, R26, R27, R29, R30, R32, R33, R34, R35: moved to B.Cu
- U3: value IS62C5128BL-45TLI -> AS6C4008A-55ZIN
- moved J8 20.6 mm to (184.9, 129.5)
- moved R29 20.6 mm to (180.7, 126.6)
- moved R32 20.6 mm to (180.7, 124.8)
- moved R34 20.6 mm to (172.1, 124.8)
- moved R35 20.6 mm to (172.1, 126.6)
- moved JP2 20.6 mm to (179.8, 119.4)
- moved R33 20.6 mm to (176.4, 126.6)
- moved R30 19.9 mm to (184.4, 126.6)
- moved JP1 17.5 mm to (162.1, 119.4)
- moved R21 17.5 mm to (162.9, 126.6)
- moved R23 17.5 mm to (167.3, 126.6)
- moved R24 17.5 mm to (162.9, 124.8)
- moved R25 17.5 mm to (158.6, 126.6)
- moved J7 17.5 mm to (167.1, 129.5)
- moved R26 17.5 mm to (154.3, 124.8), turned to 0 degrees
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Connections:
- U3 pad 1: /A17 -> /A18
- U3 pad 30: /A18 -> /A17
Routing:
- net /D4: track 0.00 -> 212.6 mm, vias 0 -> 11
- net /D7: track 0.00 -> 186.6 mm, vias 0 -> 9
- net /D5: track 0.00 -> 185.6 mm, vias 0 -> 11
- net /D3: track 0.00 -> 177.3 mm, vias 0 -> 10
- net /D6: track 0.00 -> 174.6 mm, vias 0 -> 9
- net /A1: track 0.00 -> 170.4 mm, vias 0 -> 8
- net /A0: track 0.00 -> 165.2 mm, vias 0 -> 8
- net /D2: track 0.00 -> 141.3 mm, vias 0 -> 10
- net /A7: track 0.00 -> 133.0 mm, vias 0 -> 4
- net /A6: track 0.00 -> 127.3 mm, vias 0 -> 4
- net /A5: track 0.00 -> 123.8 mm, vias 0 -> 4
- net /A4: track 0.00 -> 121.8 mm, vias 0 -> 4
- net /A2: track 0.00 -> 120.0 mm, vias 0 -> 6
- net /A3: track 0.00 -> 118.7 mm, vias 0 -> 4
- net /A12: track 0.00 -> 114.2 mm, vias 0 -> 4
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
Commit message: different path
Routing:
- net /D4: track 212.6 -> 73.3 mm, vias 11 -> 1
- net /A0: track 165.2 -> 46.4 mm, vias 8 -> 1
- net /D5: track 185.6 -> 74.6 mm, vias 11 -> 1
- net /D3: track 177.3 -> 73.3 mm, vias 10 -> 2
- net /A1: track 170.4 -> 69.9 mm, vias 8 -> 2
- net /~M1: track 104.2 -> 15.0 mm, vias 8 -> 1
- net /D6: track 174.6 -> 88.8 mm, vias 9 -> 3
- net /D7: track 186.6 -> 102.5 mm, vias 9 -> 2
- net /~RESET: track 83.0 -> 0.00 mm, vias 6 -> 0
- net /TXA: track 82.6 -> 0.00 mm, vias 2 -> 0
- net /A7: track 133.0 -> 52.8 mm, vias 4 -> 1
- net /D2: track 141.3 -> 65.7 mm, vias 10 -> 2
- net /A6: track 127.3 -> 52.7 mm, vias 4 -> 1
- net /RXA: track 73.1 -> 0.00 mm, vias 2 -> 0
- net /A5: track 123.8 -> 50.9 mm, vias 4 -> 0
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
Commit message: checkpoint
Routing:
- net /A18: track 35.2 -> 132.5 mm, vias 0 -> 4
- net /A16: track 34.3 -> 107.6 mm, vias 0 -> 2
- net /A5: track 50.9 -> 76.8 mm, vias 0 -> 2
- net /A8: track 43.3 -> 66.3 mm, vias 2 -> 4
- net /A7: track 52.8 -> 75.2 mm, vias 1 -> 2
- net /A6: track 52.7 -> 74.1 mm, vias 1 -> 2
- net /A17: track 77.1 -> 97.3 mm, vias 2 -> 4
- net /A2: track 71.4 -> 89.9 mm, vias 2 -> 4
- net /A1: track 69.9 -> 88.2 mm, vias 2 -> 4
- net /A3: track 64.0 -> 81.9 mm, vias 2 -> 4
- net /A4: track 64.4 -> 81.6 mm, vias 2 -> 4
- net /~M1: track 15.0 -> 0.00 mm, vias 1 -> 0
- net /~RFSH: track 12.6 -> 0.00 mm, vias 1 -> 0
- net /A13: track 103.6 -> 93.4 mm, vias 3 -> 4
- net /A14: track 106.3 -> 101.3 mm, vias 3 -> 4
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
Commit message: changes
Parts:
- removed R17: 10K, Resistor_SMD:R_0603_1608Metric_Pad1.05x0.95mm_HandSolder
- moved R3 16.9 mm to (186.9, 88.6)
- moved R4 13.3 mm to (186.9, 91.7), turned to 0 degrees
- moved R5 10.0 mm to (186.9, 93.2)
- moved R6 6.10 mm to (186.9, 90.2), turned to 0 degrees
- moved U2 0.57 mm to (108.5, 58.9)
Routing:
- net /D6: track 88.8 -> 253.7 mm, vias 3 -> 14
- net /D5: track 74.9 -> 223.6 mm, vias 1 -> 11
- net /D3: track 72.6 -> 205.6 mm, vias 2 -> 10
- net /D4: track 72.6 -> 204.7 mm, vias 1 -> 9
- net /A1: track 88.2 -> 215.8 mm, vias 4 -> 9
- net /D2: track 65.0 -> 192.2 mm, vias 2 -> 11
- net /A0: track 50.2 -> 172.5 mm, vias 2 -> 6
- net /D1: track 63.5 -> 178.0 mm, vias 2 -> 10
- net /D0: track 63.0 -> 174.9 mm, vias 3 -> 10
- net /D7: track 102.5 -> 209.5 mm, vias 2 -> 8
- net GND: track 0.00 -> 2.79 mm
- net VCC: track 0.00 -> 2.63 mm
- net /A2: track 89.9 -> 89.3 mm

Commit message: changed regulator, routing
Parts:
- added C32: 1uF, Capacitor_SMD:C_0603_1608Metric_Pad1.05x0.95mm_HandSolder, F.Cu at (119.1, 75.2)
- C23: value 2.2uF -> 10nF
- R13: value 100R -> 33R
- U8: moved to F.Cu
- U9: value AP7381-33SA -> LP2985-3.3; footprint Package_TO_SOT_SMD:SOT-23 -> Package_TO_SOT_SMD:SOT-23-5; moved to F.Cu
- moved U9 9.26 mm to (114.8, 76.2), turned to 0 degrees
- moved C1 6.47 mm to (116.3, 42.2)
- moved C16 2.29 mm to (148.1, 92.5), turned to 0 degrees
- moved R4 1.52 mm to (186.9, 93.2)
- moved R5 1.52 mm to (186.9, 91.7)
- moved U8 1.37 mm to (134.9, 80.5)
- turned U1 to 0 degrees
Connections:
- C23 pad 1: +3V3 -> Net-(C23-Pad1)
- U9 pad 2: +3V3 -> GND
- U9 pad 3: GND -> VCC
Routing:
- net /~RESET: track 0.00 -> 152.9 mm, vias 0 -> 10
- net /~IORQ: track 1.22 -> 141.5 mm, vias 1 -> 9
- net /~M1: track 0.00 -> 121.5 mm, vias 0 -> 10
- net /~INT: track 0.00 -> 109.1 mm, vias 0 -> 8
- net /CLK_CPU: track 0.00 -> 80.2 mm, vias 0 -> 6
- net /~RD: track 25.6 -> 95.5 mm, vias 0 -> 2
- net /CLK2: track 0.00 -> 69.4 mm, vias 0 -> 4
- net /D7: track 209.5 -> 269.3 mm, vias 8 -> 13
- net VCC: track 2.63 -> 58.7 mm, vias 0 -> 10
- net /Peripherals/IEO_0: track 0.00 -> 55.7 mm, vias 0 -> 2
- net /D5: track 223.6 -> 278.7 mm, vias 11 -> 14
- net /Peripherals/~ASTB: track 0.00 -> 53.5 mm, vias 0 -> 3
- net /Peripherals/IEO_1: track 0.00 -> 52.9 mm, vias 0 -> 4
- net /D4: track 204.7 -> 256.6 mm, vias 9 -> 12
- net /D3: track 205.6 -> 257.3 mm, vias 10 -> 13
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
Commit message: routing
Parts:
- C22, C23, C26, C27, C28: moved to F.Cu
- R3, R4, R5, R6, RN1: moved to B.Cu
- moved RN1 9.65 mm to (124.5, 59.4), turned to 90 degrees
- moved C23 7.86 mm to (115.6, 75.9)
- moved C22 6.69 mm to (112.0, 72.1)
- moved D14 5.52 mm to (111.8, 88.1), turned to 0 degrees
- moved C28 5.21 mm to (142.2, 44.5), turned to 0 degrees
- moved C32 3.78 mm to (115.6, 73.9)
- moved U9 3.17 mm to (111.9, 74.9)
- moved SW3 0.76 mm to (104.1, 66.5)
- moved C26 0.68 mm to (108.2, 73.7)
- moved C27 0.51 mm to (104.9, 73.7)
- moved R30 0.51 mm to (184.9, 126.6)
- moved U8 0.51 mm to (134.9, 80.0)
- moved D15 0.25 mm to (105.2, 92.7), turned to 0 degrees
- moved D13 0.25 mm to (134.9, 77.2)
- moved R19 0.25 mm to (134.9, 77.2)
Connections:
- U5 pad 1: /RAM_~CE -> /ROM_~CE
- U5 pad 2: /RAM_~CE -> /~WR
- U5 pad 3: Net-(D4-Pad2) -> Net-(D2-Pad1)
- U5 pad 5: /ROM_~CE -> /RAM_~CE
- U5 pad 6: /~WR -> /RAM_~CE
- U5 pad 7: Net-(D2-Pad1) -> Net-(D4-Pad2)
Routing:
- net /~WR: track 0.00 -> 156.9 mm, vias 0 -> 13
- net /~RD: track 95.5 -> 205.3 mm, vias 2 -> 7
- net /IEO: track 0.00 -> 94.9 mm, vias 0 -> 2
- net /TXA: track 0.00 -> 83.5 mm, vias 0 -> 4
- net VCC: track 58.7 -> 140.2 mm, vias 10 -> 47
- net GND: track 49.7 -> 128.5 mm, vias 12 -> 57
- net /RXA: track 0.00 -> 74.1 mm, vias 0 -> 2
- net /A0: track 182.5 -> 245.2 mm, vias 8 -> 10
- net /SIO_~CE: track 0.00 -> 62.5 mm, vias 0 -> 2
- net /~MREQ: track 0.00 -> 60.1 mm, vias 0 -> 4
- net /~PAGE: track 0.00 -> 58.5 mm, vias 0 -> 4
- net /PIO_~CE: track 0.00 -> 57.7 mm, vias 0 -> 4
- net /IDE_~CE~: track 0.00 -> 57.0 mm, vias 0 -> 1
- net /~WAIT: track 0.00 -> 56.1 mm, vias 0 -> 5
- net /IEI: track 0.00 -> 54.2 mm, vias 0 -> 2
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Other:
- board text removed: "MAX 7000S"

Commit message: cleaned up
Parts:
- added U14: 74AHCT2G04, Package_TO_SOT_SMD:SOT-363_SC-70-6_Handsoldering, B.Cu at (159.0, 55.5)
- U5: value 74LVC2G02 -> 74AHCT1G02; footprint Package_SO:TSSOP-8_3x3mm_P0.65mm -> Package_TO_SOT_SMD:SOT-353_SC-70-5_Handsoldering
- moved C9 2.29 mm to (175.5, 45.7)
- moved R8 2.29 mm to (179.1, 45.7)
- moved R9 2.16 mm to (186.1, 61.0)
- moved U5 1.73 mm to (164.0, 55.5)
- moved R11 0.89 mm to (159.1, 51.3)
- moved D3 0.88 mm to (159.1, 51.3)
- moved D2 0.76 mm to (163.2, 51.3)
- moved R10 0.76 mm to (163.2, 51.3)
- moved R12 0.76 mm to (163.2, 53.2)
- moved D4 0.75 mm to (163.2, 53.2)
- moved C10 0.51 mm to (154.9, 45.7)
Connections:
- D3 pad 2: Net-(D2-Pad1) -> Net-(D3-Pad2)
- R10 pad 1: Net-(D2-Pad2) -> GND
- R10 pad 2: VCC -> Net-(D2-Pad1)
- U5 pad 3: Net-(D2-Pad1) -> GND
- U5 pad 4: GND -> Net-(D4-Pad2)
- U5 pad 5: /RAM_~CE -> VCC
Routing:
- net /~WR: track 156.9 -> 97.9 mm, vias 13 -> 9
- net /A13: track 103.3 -> 59.4 mm, vias 4 -> 2
- net /A14: track 108.9 -> 73.6 mm, vias 4 -> 2
- net /A18: track 150.5 -> 125.0 mm, vias 6 -> 5
- net /ROM_~CE: track 24.0 -> 0.00 mm, vias 1 -> 0
- net Net-(D2-Pad1): track 16.4 -> 0.00 mm, vias 3 -> 0
- net VCC: track 140.2 -> 128.4 mm, vias 47 -> 42
- net /A3: track 130.8 -> 119.9 mm, vias 7 -> 6
- net /CPLD/LED1: track 45.7 -> 35.5 mm, vias 5 -> 4
- net Net-(D4-Pad2): track 9.51 -> 0.00 mm, vias 3 -> 0
- net /~M1: track 148.7 -> 140.8 mm, vias 12 -> 11
- net /RAM_~CE: track 10.2 -> 2.47 mm, vias 3 -> 0
- net GND: track 128.5 -> 121.0 mm, vias 57 -> 52
- net Net-(D4-Pad1): track 2.85 -> 0.00 mm, vias 1 -> 0
- net Net-(D3-Pad1): track 2.82 -> 0.00 mm, vias 1 -> 0
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
Commit message: routing
Parts:
- moved D4 0.13 mm to (163.2, 53.1)
- moved R12 0.13 mm to (163.2, 53.1), turned to 180 degrees
Routing:
- net /~WR: track 97.9 -> 169.3 mm, vias 9 -> 13
- net /ROM_~CE: track 0.00 -> 60.0 mm, vias 0 -> 6
- net /CPLD/USER_PB: track 11.9 -> 62.8 mm, vias 2 -> 4
- net /CPLD/SW1: track 6.97 -> 55.8 mm, vias 1 -> 4
- net /CPLD/SW0: track 7.91 -> 50.5 mm, vias 1 -> 4
- net /CPLD/SW5: track 7.91 -> 49.6 mm, vias 1 -> 4
- net /CPLD/SW3: track 6.35 -> 47.8 mm, vias 1 -> 3
- net /CPLD/SW4: track 6.97 -> 45.1 mm, vias 1 -> 4
- net /CPLD/LED2: track 0.00 -> 37.6 mm, vias 0 -> 2
- net /CPLD/SW2: track 6.35 -> 41.1 mm, vias 1 -> 3
- net GND: track 121.0 -> 148.3 mm, vias 52 -> 60
- net /RAM_~CE: track 2.47 -> 29.6 mm, vias 0 -> 3
- net /A14: track 73.6 -> 98.4 mm, vias 2 -> 4
- net /A13: track 59.4 -> 83.8 mm, vias 2 -> 4
- net VCC: track 128.4 -> 147.2 mm, vias 42 -> 48
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