File: power.sch (KiCad schematic (older format))
At the start: 16 parts, among them J10 USB_B_Micro, J9 Jack-DC, U12 MAX40203AUK, U13 MAX40203AUK

Commit message: do over with additional pmod
Parts:
- removed C27, C32, C33: 100nF, Capacitor_SMD:C_0603_1608Metric_Pad1.05x0.95mm_HandSolder, symbol Device:C_Small
- removed C28, C29: 100uF, Capacitor_SMD:C_1206_3216Metric_Pad1.42x1.75mm_HandSolder, symbol Device:C_Small
- removed C30, C31, C34, C35: 2.2uF, Capacitor_SMD:C_0603_1608Metric_Pad1.05x0.95mm_HandSolder, symbol Device:C_Small
- removed D11: Blue, LED_SMD:LED_0603_1608Metric_Pad1.05x0.95mm_HandSolder, symbol THS-80-rescue:LED-Device-max_breakout-rescue-sbc_z80-rescue
- removed J10: USB_B_Micro, Connector_USB:USB_Micro-B_Amphenol_10103594-0001LF_Horizontal, symbol Connector:USB_B_Micro
- removed R19: 1M, Resistor_SMD:R_0603_1608Metric_Pad1.05x0.95mm_HandSolder, symbol Device:R_Small
- removed R20: 360R, Resistor_SMD:R_0603_1608Metric_Pad1.05x0.95mm_HandSolder, symbol Device:R_Small
- removed U12, U13: MAX40203AUK, Package_TO_SOT_SMD:SOT-23-5_HandSoldering, symbol Analog_Switch:MAX40200AUK
- added C13, C5: 10nF, Capacitor_SMD:C_0603_1608Metric_Pad1.05x0.95mm_HandSolder, symbol Device:C_Small
- added C15, C3, C6, C7, C9: 1uF, Capacitor_SMD:C_0603_1608Metric_Pad1.05x0.95mm_HandSolder, symbol Device:C_Small
- added C8: 4.7uF, Capacitor_SMD:C_0603_1608Metric_Pad1.05x0.95mm_HandSolder, symbol Device:C_Small
- added D1: BAT54W, Diode_SMD:D_SOD-123, symbol Device:D_Schottky_Small
- added D2: BLU, LED_SMD:LED_0603_1608Metric_Pad1.05x0.95mm_HandSolder, symbol Device:LED
- added FB1: 100R @ 100Mhz, Capacitor_SMD:C_0603_1608Metric_Pad1.05x0.95mm_HandSolder, symbol Device:Ferrite_Bead_Small
- added J4: USB_B_Micro, Connector_USB:USB_Micro-B_Amphenol_10103594-0001LF_Horizontal, symbol max_breakout-rescue:USB_B_Micro-Connector
- added R4, R7: 100K, Resistor_SMD:R_0603_1608Metric_Pad1.05x0.95mm_HandSolder, symbol Device:R_Small
- added R5: 20K, Resistor_SMD:R_0603_1608Metric_Pad1.05x0.95mm_HandSolder, symbol Device:R_Small
- added R6, R8: 1K, Resistor_SMD:R_0603_1608Metric_Pad1.05x0.95mm_HandSolder, symbol Device:R_Small
- added U2: LP2985-5.0, Package_TO_SOT_SMD:SOT-23-5, symbol Regulator_Linear:LP2985-5.0
- added U4: TPS2113A, Package_SO:TSSOP-8_4.4x3mm_P0.65mm, symbol max_breakout-rescue:TPS2113A-Power_Management
- added U5: LP2985-3.3, Package_TO_SOT_SMD:SOT-23-5, symbol Regulator_Linear:LP2985-3.3
Connections:
- net GND: now also C13.2, C15.2, C3.2, C5.2, C6.2, C7.2, C8.2, C9.2, J4.4 (ID), J4.5 (GND), R4.2, R5.2, R6.2, R8.2, U2.2 (GND), U4.5 (GND), U5.2 (GND)
- net at J9.1: now also D1.2 (A)
- new net: C6.1, J4.1 (VBUS), U4.8 (IN1)
- new net: C3.1, FB1.1, U2.1 (VIN), U2.3 (ON/~OFF~)
- new net: C5.1, U2.4 (BP)
- new net: C7.1, U2.5 (VOUT), U4.6 (IN2)
- new net: C13.1, U5.4 (BP)
- new net: D1.1 (K), FB1.2
- new net: R7.2, U4.1 (STAT)
- new net: R4.1, U4.2 (~EN)
- new net: R5.1, U4.3 (VSNS)
- new net: R6.1, U4.4 (ILIM)
- new net: D2.1 (K), R8.1
- new net +3V3: C15.1, U5.5 (VOUT)
- new net +5V: C8.1, C9.1, D2.2 (A), R7.1, U4.7 (OUT), U5.1 (VIN), U5.3 (ON/~OFF~)
- no-connect marks 2 -> 3
Other:
- moved on the sheet: J9
